File: hardware/business-card.kicad_sch (KiCad schematic)
At the start: 26 parts, among them J1 SWD, J2 USB_A_PCB_Edge_receptacle, SW1 BTN_UP, SW2 BTN_DOWN, SW3 BTN_LEFT, SW4 BTN_RIGHT, SW5 RST, SW6 BTN_A, SW7 BTN_B, U1 STM32G030F6Px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

Commit message: hardware: Consistent label numbering
Number the button matrix labels from top to bottom to match the
numbering of the LED matrix.

The labels on the MCU pins have been changed accordingly, so that
this change is a no-op.

The PCB has been updated accordingly, but other than netlist names
nothing has changed.
Connections:
- net BM1: now also R1.1, U1.1 (PB7/PB8); no longer R3.1, U1.15 (PB0/PB1/PB2/PA8)
- net BM3: now also R3.1, U1.15 (PB0/PB1/PB2/PA8); no longer R1.1, U1.1 (PB7/PB8)
Changed lines of the file:
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@@
 		)
 	)
-	(label "BM1"
+	(label "BM3"
 		(at 29.21 44.45 180)
 		(fields_autoplaced yes)
@@
 		)
 	)
-	(label "BM3"
+	(label "BM1"
 		(at 97.79 99.06 180)
 		(fields_autoplaced yes)
@@
 		)
 	)
+	(label "BM3"
+		(at 97.79 121.92 180)
+		(fields_autoplaced yes)
+		(effects
+			(font
+				(size 1.27 1.27)
+			)
+			(justify right bottom)
+		)
+	)
 	(label "BM1"
-		(at 97.79 121.92 180)
-		(fields_autoplaced yes)
-		(effects
-			(font
-				(size 1.27 1.27)
-			)
-			(justify right bottom)
-		)
-	)
-	(label "BM3"
 		(at 29.21 49.53 180)
 		(fields_autoplaced yes)
