File: hardware/business-card.kicad_pcb (KiCad board)
At the start: 2 copper layers, 88.9 x 50.8 mm, 127 parts, among them J1 SWD, J2 USB_A_PCB_Edge_receptacle, SW1 BTN_UP, SW2 BTN_DOWN, SW3 BTN_LEFT, SW4 BTN_RIGHT, SW5 RST, SW6 BTN_A, SW7 BTN_B, U1 STM32G030F6Px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

Commit message: hardware: Consistent label numbering
Number the button matrix labels from top to bottom to match the
numbering of the LED matrix.

The labels on the MCU pins have been changed accordingly, so that
this change is a no-op.

The PCB has been updated accordingly, but other than netlist names
nothing has changed.
Connections:
- R1 pad 1: /BM3 -> /BM1
- R3 pad 1: /BM1 -> /BM3
- U1 pad 1: /BM3 -> /BM1
- U1 pad 15: /BM1 -> /BM3
Routing:
- net /BM3: track 10.8 -> 10.0 mm
- net /BM1: track 10.0 -> 10.8 mm
Changed lines of the file:
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@@
 			(layers "F.Cu" "F.Paste" "F.Mask")
 			(roundrect_rratio 0.25)
-			(net 33 "/BM3")
+			(net 35 "/BM1")
 			(pinfunction "PB7/PB8")
 			(pintype "bidirectional")
@@
 			(layers "F.Cu" "F.Paste" "F.Mask")
 			(roundrect_rratio 0.25)
-			(net 35 "/BM1")
+			(net 33 "/BM3")
 			(pinfunction "PB0/PB1/PB2/PA8")
 			(pintype "bidirectional")
@@
 			(layers "F.Cu" "F.Paste" "F.Mask")
 			(roundrect_rratio 0.25)
-			(net 35 "/BM1")
+			(net 33 "/BM3")
 			(pintype "passive")
 		)
@@
 			(layers "F.Cu" "F.Paste" "F.Mask")
 			(roundrect_rratio 0.25)
-			(net 33 "/BM3")
+			(net 35 "/BM1")
 			(pintype "passive")
 		)
@@
 	)
 	(segment
-		(start 47.4363 54.1175)
-		(end 47.851 53.7028)
+		(start 53.665 49.8679)
+		(end 53.665 49.2075)
 		(width 0.2)
 		(layer "F.Cu")
@@
 	)
 	(segment
-		(start 45.72 49.53)
-		(end 44.9992 50.2508)
+		(start 50.6186 52.9143)
+		(end 53.665 49.8679)
 		(width 0.2)
 		(layer "F.Cu")
@@
 	)
 	(segment
-		(start 47.851 53.7028)
-		(end 49.1853 53.7028)
+		(start 46.1457 52.9143)
+		(end 50.6186 52.9143)
 		(width 0.2)
 		(layer "F.Cu")
@@
 	)
 	(segment
-		(start 49.1853 53.7028)
-		(end 50.415 54.9325)
+		(start 45.72 53.34)
+		(end 46.1457 52.9143)
 		(width 0.2)
 		(layer "F.Cu")
@@
 	)
 	(segment
-		(start 44.9992 53.8049)
-		(end 45.3118 54.1175)
+		(start 47.9475 49.2075)
+		(end 45.72 51.435)
 		(width 0.2)
 		(layer "F.Cu")
-		(net 33)
+		(net 34)
 	)
 	(segment
-		(start 45.3118 54.1175)
-		(end 47.4363 54.1175)
+		(start 50.415 49.2075)
+		(end 47.9475 49.2075)
 		(width 0.2)
 		(layer "F.Cu")
-		(net 33)
+		(net 34)
 	)
 	(segment
-		(start 44.9992 50.2508)
-		(end 44.9992 53.8049)
+		(start 47.4363 54.1175)
+		(end 47.851 53.7028)
 		(width 0.2)
 		(layer "F.Cu")
-		(net 33)
+		(net 35)
 	)
 	(segment
-		(start 47.9475 49.2075)
-		(end 45.72 51.435)
+		(start 45.72 49.53)
+		(end 44.9992 50.2508)
 		(width 0.2)
 		(layer "F.Cu")
-		(net 34)
+		(net 35)
 	)
 	(segment
-		(start 50.415 49.2075)
-		(end 47.9475 49.2075)
+		(start 47.851 53.7028)
+		(end 49.1853 53.7028)
 		(width 0.2)
 		(layer "F.Cu")
-		(net 34)
+		(net 35)
 	)
 	(segment
-		(start 53.665 49.8679)
-		(end 53.665 49.2075)
+		(start 49.1853 53.7028)
+		(end 50.415 54.9325)
 		(width 0.2)
 		(layer "F.Cu")
@@
 	)
 	(segment
-		(start 50.6186 52.9143)
-		(end 53.665 49.8679)
+		(start 44.9992 53.8049)
+		(end 45.3118 54.1175)
 		(width 0.2)
 		(layer "F.Cu")
@@
 	)
 	(segment
-		(start 46.1457 52.9143)
-		(end 50.6186 52.9143)
+		(start 45.3118 54.1175)
+		(end 47.4363 54.1175)
 		(width 0.2)
 		(layer "F.Cu")
@@
 	)
 	(segment
-		(start 45.72 53.34)
-		(end 46.1457 52.9143)
+		(start 44.9992 50.2508)
+		(end 44.9992 53.8049)
 		(width 0.2)
 		(layer "F.Cu")

Commit message: hardware: add panelization
Parts:
- added REF**: Tab, PCM_kikit:Tab, F.Cu at (12.7, 20.3)
- added REF**: Tab, PCM_kikit:Tab, F.Cu at (101.6, 55.9)
- added REF**: Tab, PCM_kikit:Tab, F.Cu at (101.6, 43.2)
- added REF**: Tab, PCM_kikit:Tab, F.Cu at (12.7, 55.9)
