File: hardware/led_matrix.kicad_sch (KiCad schematic)
At the start: 100 parts

Commit message: hardware: add panelization
Parts:
- D10, D11, D12, D13, D14, D15, D16, D17, D18, D19, D20, D21, D22, D23, D24, D25, D26, D27, D28, D29, D30, D31, D32, D33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: LCSC C2286 -> (none); MPN (none) -> C2286
- R10, R11, R12, R13, R4, R5, R6, R7, R8, R9: LCSC C4275 -> (none); MPN (none) -> C4275
